File: PCB/lightmeter.kicad_pcb (KiCad board)
At the start: 2 copper layers, 43.2 x 68.6 mm, 17 parts, among them J2 TSL2561, J3 BabySitter, J4 SYSOFF, Q1 2N3904, SW2 DOWN, SW3 UP, U1 Teensy3.2, U2 ENCODER_2LED

Commit message: PCB
Routing:
- net GND: track 158.1 -> 142.2 mm
- net ENC_B: track 53.3 -> 38.5 mm
- net Net-(C1-Pad1): track 77.3 -> 68.9 mm
- net /VOUT+: track 32.9 -> 25.1 mm
- net ENC_A: track 40.9 -> 47.5 mm
- net SW_ROT: track 30.0 -> 28.1 mm, vias 2 -> 0
- net Net-(Q1-Pad2): track 18.3 -> 16.8 mm
- net Net-(D3-Pad1): track 34.5 -> 33.2 mm
- net LED_G: track 27.4 -> 28.4 mm
- net LED_R: track 23.1 -> 22.1 mm
- added copper zone on B.Cu, net GND
- added copper zone on F.Cu, net GND
Other:
- board text added: "GND"
- board text added: "SCL"
- board text added: "SDA"
- board text added: "Teensy Light Meter"
- board text added: "VOUT+"
- board text added: "Vpu"
- board text added: "ignore pads"
- board text added: "x"
